Commit message: add imu_driver & keyboard

File: mick_description/urdf/mickX4.urdf (robot description, URDF)
Before this commit: robot smartcar, 14 links, 13 joints
Links:
- removed link laser
- added link rslidar; visual cylinder length=.0826 radius=0.0487
Joints:
- joint laser_joint: child laser -> rslidar

Commit message: add mickx4 gmapping

File: mick_description/urdf/mickX4.urdf (robot description, URDF)
Before this commit: robot smartcar, 14 links, 13 joints
Links:
- added link body; visual box size=0.66 .54 .1
- link base_link: geometry visual box size=0.01 .01 .01
- link camera: geometry visual mesh filename=package://mick_description/urdf/mesh/ZED.stl scale=0.001 0.001 0.001
- link left_back_wheel: geometry visual mesh filename=package://mick_description/urdf/mesh/wheel.stl scale=0.001 0.001 0.001
- link left_front_wheel: geometry visual mesh filename=package://mick_description/urdf/mesh/wheel.stl scale=0.001 0.001 0.001
- link right_back_wheel: geometry visual mesh filename=package://mick_description/urdf/mesh/wheel.stl scale=0.001 0.001 0.001
- link right_front_wheel: geometry visual mesh filename=package://mick_description/urdf/mesh/wheel.stl scale=0.001 0.001 0.001
- link rslidar: geometry visual mesh filename=package://mick_description/urdf/mesh/RS-LiDAR-16.stl scale=0.001 0.001 0.001
Joints:
- added joint body: type continuous, parent base_link, child body, origin xyz=0.0 0.0 0.14 rpy=0 0 0, axis 0 0 1, limit effort=100 velocity=100
- joint camera: origin xyz=0.17 0.0 0.62 -> xyz=0.17 0.0 0.75
- joint laser_joint: origin xyz=0.0 0.0 0.66 -> xyz=0.0 0.0 0.80 rpy=0 0 0
- joint left_back_wheel_joint: origin xyz=-0.22 0.31 0 rpy=1.57075 0 0 -> xyz=-0.35 0.285 0 rpy=1.57075 0 0
- joint left_front_wheel_joint: origin xyz=0.22 0.31 0 rpy=1.57075 0 0 -> xyz=0.1 0.285 0 rpy=1.57075 0 0
- joint part1_joint: parent base_link -> body
- joint part2_joint: parent base_link -> body
- joint part3_joint: parent base_link -> body
- joint part4_joint: parent base_link -> body
- joint part5_joint: parent base_link -> body
- joint part6_joint: parent base_link -> body
- joint part7_joint: parent base_link -> body
- joint right_back_wheel_joint: origin xyz=-0.22 -0.31 0 rpy=1.57075 0 0 -> xyz=-0.35 -0.37 0 rpy=1.57075 0 0
- joint right_front_wheel_joint: origin xyz=0.22 -0.31 0 rpy=1.57075 0 0 -> xyz=0.1 -0.37 0 rpy=1.57075 0 0

Commit message: turning parameters for gmapping

File: mick_description/urdf/mickX4.urdf (robot description, URDF)
Before this commit: robot mickx4, 15 links, 14 joints
Links:
- link rslidar: geometry visual cylinder length=.0826 radius=0.0487
Joints:
- joint laser_joint: type fixed -> continuous
- joint part1_joint: type fixed -> continuous
- joint part2_joint: type fixed -> continuous
- joint part3_joint: type fixed -> continuous
- joint part4_joint: type fixed -> continuous

Commit message: add cartographer node

File: mick_description/urdf/mickX4.urdf (robot description, URDF)
Before this commit: robot mickx4, 15 links, 14 joints
Joints:
- removed joint laser_joint
- added joint rslidar_joint: type fixed, parent base_link, child rslidar, origin xyz=0.0 0.0 0.80 rpy=0 0 0
- joint body: type continuous -> fixed
- joint left_back_wheel_joint: origin xyz=-0.35 0.285 0 rpy=1.57075 0 0 -> xyz=-0.35 0.285 -0.14 rpy=1.57075 0 0; parent base_link -> body; type continuous -> fixed
- joint left_front_wheel_joint: origin xyz=0.1 0.285 0 rpy=1.57075 0 0 -> xyz=0.1 0.285 -0.14 rpy=1.57075 0 0; parent base_link -> body; type continuous -> fixed
- joint part1_joint: type continuous -> fixed
- joint part2_joint: type continuous -> fixed
- joint part3_joint: type continuous -> fixed
- joint part4_joint: type continuous -> fixed
- joint right_back_wheel_joint: origin xyz=-0.35 -0.37 0 rpy=1.57075 0 0 -> xyz=-0.35 -0.37 -0.14 rpy=1.57075 0 0; parent base_link -> body; type continuous -> fixed
- joint right_front_wheel_joint: origin xyz=0.1 -0.37 0 rpy=1.57075 0 0 -> xyz=0.1 -0.37 -0.14 rpy=1.57075 0 0; parent base_link -> body; type continuous -> fixed

Commit message: add cartographer 3D

File: mick_description/urdf/mickX4.urdf (robot description, URDF)
Before this commit: robot mickx4, 15 links, 14 joints
Links:
- added link imu_link; visual box size=.05 .02 .02
Joints:
- removed joint camera
- added joint camera_joint: type fixed, parent base_link, child camera, origin xyz=0.17 0.0 0.75
- added joint imu_link_joint: type fixed, parent base_link, child imu_link, origin xyz=0.05 0.0 0.75

Commit message: add Lego-LOAM node

File: mick_description/urdf/mickX4.urdf (robot description, URDF)
Before this commit: robot mickx4, 16 links, 15 joints
Links:
- added link base_footprint
Joints:
- added joint base_joint: type fixed, parent base_footprint, child base_link, origin xyz=0.0 0.0 0.01

Commit message: fix navigation parameters

File: mick_description/urdf/mickX4.urdf (robot description, URDF)
Before this commit: robot mickx4, 17 links, 16 joints
Joints:
- joint base_joint: child base_link -> base_footprint; origin xyz=0.0 0.0 0.01 -> xyz=0.0 0.0 -0.01; parent base_footprint -> base_link
