Commit message: Navigation simulation

File: mickrobot_description/urdf/mickrobot_stl_rviz.urdf (robot description, URDF)
Before this commit: robot mickrobot, 10 links, 9 joints
Links:
- added link base_footprint; visual sphere radius=0.001
- link base_link: geometry collision box size=0.333 0.6 0.16; visual mesh filename=package://mickrobot_description/urdf/mesh/mickx4_body1.STL scale=0.001 0.001 0.001
- link sensor_link: geometry collision mesh filename=package://mickrobot_description/urdf/mesh/mickx4_sensorkit1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 scale=0.001 0.001 0.001; visual mesh filename=package://mickrobot_description/urdf/mesh/mickx4_sensorkit1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 scale=0.001 0.001 0.001
Joints:
- added joint base_joint: type fixed, parent base_footprint, child base_link, origin xyz=-0.3 -0.1665 0.0 rpy=0 0 0
- joint camera_joint: origin xyz=0.1665 0.025 0.15 rpy=0 0 -1.57079 -> xyz=0.53 0.16 0.15 rpy=0 0 0
- joint gnss_joint: origin xyz=0.173 0.165 0.25 rpy=0.0 0.0 0.0 -> xyz=0.40 0.165 0.25 rpy=0.0 0.0 0.0
- joint imu_joint: origin xyz=0.173 0.165 0.163 rpy=0.0 0.0 3.14159 -> xyz=0.40 0.165 0.163 rpy=0.0 0.0 0.0
- joint laser_joint: origin xyz=0.173 0.13 0.37 -> xyz=0.42 0.16 0.37
- joint left_back_wheel_joint: origin xyz=-0.027 0.1 0 -> xyz=0.1 0.32 -0.03
- joint left_front_wheel_joint: origin xyz=-0.027 0.5 0 -> xyz=0.49 0.32 -0.03
- joint right_back_wheel_joint: origin xyz=0.36 0.1 0 -> xyz=0.50 -0.02 -0.03
- joint right_front_wheel_joint: origin xyz=0.36 0.5 0 -> xyz=0.1 -0.02 -0.03
- joint sensor_joint: origin xyz=0.29 0.20 0.15 -> xyz=0.29 0.05 0.15

File: mickrobot_description/urdf/mickrobot_stl（复件）.urdf (robot description, URDF)
Before this commit: robot mickrobot, 11 links, 10 joints
Links:
- removed link base_footprint
- link base_link: geometry collision box size=0.48 0.32 0.111; visual mesh filename=/home/liiujinjian/ros2_ws/src/mick_robot/mickrobot_descript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 scale=0.001 0.001 0.001
- link laser_link: mass 0.5 -> 0.1; geometry collision cylinder length=0.05 radius=0.04; visual cylinder length=0.05 radius=0.04
Joints:
- removed joint base_joint
- joint right_back_wheel_joint: origin xyz=0.1 -0.02 0 -> xyz=0.50 -0.02 0
- joint right_front_wheel_joint: origin xyz=0.50 -0.02 0 -> xyz=0.1 -0.02 0

Commit message: modify gazebo stl

File: mickrobot_description/urdf/mickrobot_stl_rviz.urdf (robot description, URDF)
Before this commit: robot mickrobot, 11 links, 10 joints
Links:
- removed link left_back_wheel
- removed link left_front_wheel
- removed link right_front_wheel
- link base_link: geometry collision box size=0.6 0.333 0.16; visual mesh filename=package://mickrobot_description/urdf/mesh/mickx4_body.STL scale=0.001 0.001 0.001
- link camera_link: geometry collision box size=0.2 0.09 0.03; visual box size=0.02 0.09 0.03
- link imu_link: geometry collision box size=0.07 0.07 0.02; visual box size=0.07 0.07 0.02
- link sensor_link: geometry collision mesh filename=package://mickrobot_description/urdf/mesh/mickx4_sensorkit.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 scale=0.001 0.001 0.001; visual mesh filename=package://mickrobot_description/urdf/mesh/mickx4_sensorkit1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 scale=0.001 0.001 0.001
Joints:
- removed joint left_back_wheel_joint
- removed joint left_front_wheel_joint
- removed joint right_front_wheel_joint
- joint base_joint: origin xyz=-0.3 -0.1665 0.0 rpy=0 0 0 -> xyz=0.0 0.0 0.0 rpy=0 0 0
- joint camera_joint: origin xyz=0.53 0.16 0.15 rpy=0 0 0 -> xyz=0.29 0.0 0.15 rpy=0 0 0
- joint gnss_joint: origin xyz=0.40 0.165 0.25 rpy=0.0 0.0 0.0 -> xyz=0.235 0.0 0.42 rpy=0.0 0.0 0.0
- joint imu_joint: origin xyz=0.40 0.165 0.163 rpy=0.0 0.0 0.0 -> xyz=0.23 0.0 0.27 rpy=0.0 0.0 0.0
- joint laser_joint: origin xyz=0.42 0.16 0.37 -> xyz=0.23 0.0 0.38
- joint right_back_wheel_joint: origin xyz=0.50 -0.02 -0.03 -> xyz=-0.2 -0.24 0.0
- joint sensor_joint: origin xyz=0.29 0.05 0.15 -> xyz=0.09 -0.1165 0.16

Commit message: modify mickrobot_stl_rviz.urdf

File: mickrobot_description/urdf/mickrobot_stl_rviz.urdf (robot description, URDF)
Before this commit: robot mickrobot, 8 links, 7 joints
Links:
- added link left_back_wheel, mass 1; collision cylinder length=0.06 radius=0.1016; visual mesh filename=package://mickrobot_description/urdf/mesh/mickx4_wheel_8inc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 scale=0.001 0.001 0.001
- added link left_front_wheel, mass 1; collision cylinder length=0.06 radius=0.1016; visual mesh filename=package://mickrobot_description/urdf/mesh/mickx4_wheel_8inc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 scale=0.001 0.001 0.001
- added link right_front_wheel, mass 1; collision cylinder length=0.06 radius=0.1016; visual mesh filename=package://mickrobot_description/urdf/mesh/mickx4_wheel_8inc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 scale=0.001 0.001 0.001
Joints:
- added joint left_back_wheel_joint: type continuous, parent base_link, child left_back_wheel, origin xyz=-0.2 0.24 0.0, axis 1 0 0, limit effort=100 velocity=100
- added joint left_front_wheel_joint: type continuous, parent base_link, child left_front_wheel, origin xyz=0.2 0.24 0.0, axis 1 0 0, limit effort=100 velocity=100
- added joint right_front_wheel_joint: type continuous, parent base_link, child right_front_wheel, origin xyz=0.2 -0.24 0.0, axis 1 0 0, limit effort=100 velocity=100
