Commit message: 添加模型

File: mickrobot_description/urdf/mickrobot_stl.urdf (robot description, URDF)
Before this commit: robot mickrobot, 1 links, 0 joints
Links:
- added link camera_link, mass 0.1; collision box size=0.05 0.05 0.05; visual box size=0.05 0.05 0.05
- added link gnss_link, mass 0.5; collision box size=0.02 0.02 0.02; visual box size=0.02 0.02 0.02
- added link imu_link, mass 0.5; collision box size=0.02 0.02 0.02; visual box size=0.02 0.02 0.02
- added link laser_link, mass 0.1; collision cylinder length=0.05 radius=0.04; visual cylinder length=0.05 radius=0.04
- added link left_back_wheel, mass 1; collision cylinder length=0.06 radius=0.1016; visual mesh filename=/home/wyt/mickrobot_ws/src/mickrobot_description/urdf/mesh/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 scale=0.001 0.001 0.001
- added link left_front_wheel, mass 1; collision cylinder length=0.06 radius=0.1016; visual mesh filename=/home/wyt/mickrobot_ws/src/mickrobot_description/urdf/mesh/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 scale=0.001 0.001 0.001
- added link right_back_wheel, mass 1; collision cylinder length=0.06 radius=0.1016; visual mesh filename=/home/wyt/mickrobot_ws/src/mickrobot_description/urdf/mesh/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 scale=0.001 0.001 0.001
- added link right_front_wheel, mass 1; collision cylinder length=0.06 radius=0.1016; visual mesh filename=/home/wyt/mickrobot_ws/src/mickrobot_description/urdf/mesh/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 scale=0.001 0.001 0.001
- added link sensor_link, mass 1; collision mesh filename=/home/wyt/mickrobot_ws/src/mickrobot_description/urdf/mesh/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 scale=0.001 0.001 0.001; visual mesh filename=/home/wyt/mickrobot_ws/src/mickrobot_description/urdf/mesh/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 scale=0.001 0.001 0.001
- link base_link: mass 25.00 -> 25; geometry collision box size=0.333 0.6 0.16; visual mesh filename=/home/wyt/mickrobot_ws/src/mickrobot_description/urdf/mesh/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 scale=0.001 0.001 0.001
Joints:
- added joint camera_joint: type fixed, parent base_link, child camera_link, origin xyz=0.1665 0.025 0.15 rpy=0 0 -1.57079
- added joint gnss_joint: type fixed, parent base_link, child gnss_link, origin xyz=0.173 0.165 0.25 rpy=0.0 0.0 0.0
- added joint imu_joint: type fixed, parent base_link, child imu_link, origin xyz=0.173 0.165 0.163 rpy=0.0 0.0 3.14159
- added joint laser_joint: type fixed, parent base_link, child laser_link, origin xyz=0.173 0.13 0.37
- added joint left_back_wheel_joint: type continuous, parent base_link, child left_back_wheel, origin xyz=-0.027 0.1 0, axis 1 0 0, limit effort=100 velocity=100
- added joint left_front_wheel_joint: type continuous, parent base_link, child left_front_wheel, origin xyz=-0.027 0.5 0, axis 1 0 0, limit effort=100 velocity=100
- added joint right_back_wheel_joint: type continuous, parent base_link, child right_back_wheel, origin xyz=0.36 0.1 0, axis 1 0 0, limit effort=100 velocity=100
- added joint right_front_wheel_joint: type continuous, parent base_link, child right_front_wheel, origin xyz=0.36 0.5 0, axis 1 0 0, limit effort=100 velocity=100
- added joint sensor_joint: type fixed, parent base_link, child sensor_link, origin xyz=0.29 0.20 0.15

Commit message: fix coordinate system

File: mickrobot_description/urdf/mickrobot_stl.urdf (robot description, URDF)
Before this commit: robot mickrobot, 11 links, 10 joints
Links:
- link base_link: geometry collision box size=0.6 0.333 0.16; visual mesh filename=/home/mickrobot/ros2_mick_ws/src/mick_robot/mickrobot_descr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 scale=0.001 0.001 0.001
- link camera_link: geometry collision box size=0.2 0.09 0.03; visual box size=0.02 0.09 0.03
- link imu_link: geometry collision box size=0.07 0.07 0.02; visual box size=0.07 0.07 0.02
- link laser_link: mass 0.5 -> 0.1; geometry collision cylinder length=0.05 radius=0.04; visual cylinder length=0.05 radius=0.04
- link left_back_wheel: geometry collision cylinder length=0.06 radius=0.1016; visual mesh filename=/home/mickrobot/ros2_mick_ws/src/mick_robot/mickrobot_descr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 scale=0.001 0.001 0.001
- link left_front_wheel: geometry collision cylinder length=0.06 radius=0.1016; visual mesh filename=/home/mickrobot/ros2_mick_ws/src/mick_robot/mickrobot_descr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 scale=0.001 0.001 0.001
- link right_back_wheel: geometry collision cylinder length=0.06 radius=0.1016; visual mesh filename=/home/mickrobot/ros2_mick_ws/src/mick_robot/mickrobot_descr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 scale=0.001 0.001 0.001
- link right_front_wheel: geometry collision cylinder length=0.06 radius=0.1016; visual mesh filename=/home/mickrobot/ros2_mick_ws/src/mick_robot/mickrobot_descr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 scale=0.001 0.001 0.001
- link sensor_link: geometry collision box size=0.09 0.12 0.20; visual mesh filename=/home/mickrobot/ros2_mick_ws/src/mick_robot/mickrobot_descr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 scale=0.001 0.001 0.001
Joints:
- joint base_joint: origin xyz=-0.3 -0.15 0.10159885920454641 rpy=0 0 0 -> xyz=0.0 0.0 0.0 rpy=0 0 0
- joint camera_joint: origin xyz=0.53 0.16 0.15 rpy=0 0 0 -> xyz=0.29 0.0 0.31 rpy=0 0 0
- joint gnss_joint: origin xyz=0.40 0.165 0.25 rpy=0.0 0.0 0.0 -> xyz=0.235 0.0 0.42 rpy=0.0 0.0 0.0
- joint imu_joint: origin xyz=0.40 0.165 0.163 rpy=0.0 0.0 0.0 -> xyz=0.23 0.0 0.27 rpy=0.0 0.0 0.0
- joint laser_joint: origin xyz=0.42 0.16 0.37 -> xyz=0.23 0.0 0.38
- joint left_back_wheel_joint: origin xyz=0.1 0.32 0 -> xyz=-0.2 0.26 0.0
- joint left_front_wheel_joint: origin xyz=0.50 0.32 0 -> xyz=0.2 0.26 0.0
- joint right_back_wheel_joint: origin xyz=0.1 -0.02 0 -> xyz=-0.2 -0.26 0.0
- joint right_front_wheel_joint: origin xyz=0.50 -0.02 0 -> xyz=0.2 -0.26 0.0
- joint sensor_joint: origin xyz=0.29 0.05 0.15 -> xyz=0.09 -0.1165 0.16

File: mickrobot_description/urdf/mickrobot_stl_rviz.urdf (robot description, URDF)
Before this commit: robot mickrobot, 11 links, 10 joints
Links:
- link camera_link: geometry collision box size=0.02 0.09 0.03; visual box size=0.02 0.09 0.03
- link sensor_link: geometry collision box size=0.09 0.12 0.20; visual mesh filename=package://mickrobot_description/urdf/mesh/mickx4_sensorkit1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 scale=0.001 0.001 0.001
Joints:
- joint camera_joint: origin xyz=0.29 0.0 0.15 rpy=0 0 0 -> xyz=0.29 0.0 0.31 rpy=0 0 0
- joint left_back_wheel_joint: origin xyz=-0.2 0.24 0.0 -> xyz=-0.2 0.26 0.0
- joint left_front_wheel_joint: origin xyz=0.2 0.24 0.0 -> xyz=0.2 0.26 0.0
- joint right_back_wheel_joint: origin xyz=-0.2 -0.24 0.0 -> xyz=-0.2 -0.26 0.0
- joint right_front_wheel_joint: origin xyz=0.2 -0.24 0.0 -> xyz=0.2 -0.26 0.0

Commit message: 修改gazebo urdf文件

File: mickrobot_description/urdf/mickrobot_stl.urdf (robot description, URDF)
Before this commit: robot mickrobot, 11 links, 10 joints
Links:
- link base_link: geometry collision box size=0.6 0.333 0.16; visual mesh filename=/home/crp/ros2_ws/src/mick_robot/mickrobot_description/urdf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 scale=0.001 0.001 0.001
- link left_back_wheel: geometry collision cylinder length=0.06 radius=0.1016; visual mesh filename=/home/crp/ros2_ws/src/mick_robot/mickrobot_description/urdf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 scale=0.001 0.001 0.001
- link left_front_wheel: geometry collision cylinder length=0.06 radius=0.1016; visual mesh filename=/home/crp/ros2_ws/src/mick_robot/mickrobot_description/urdf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 scale=0.001 0.001 0.001
- link right_back_wheel: geometry collision cylinder length=0.06 radius=0.1016; visual mesh filename=/home/crp/ros2_ws/src/mick_robot/mickrobot_description/urdf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 scale=0.001 0.001 0.001
- link right_front_wheel: geometry collision cylinder length=0.06 radius=0.1016; visual mesh filename=/home/crp/ros2_ws/src/mick_robot/mickrobot_description/urdf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 scale=0.001 0.001 0.001
- link sensor_link: geometry collision box size=0.09 0.12 0.20; visual mesh filename=/home/crp/ros2_ws/src/mick_robot/mickrobot_description/urdf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 scale=0.001 0.001 0.001

Commit message: modify gazebo 3d launch

File: mickrobot_description/urdf/mickrobot_stl.urdf (robot description, URDF)
Before this commit: robot mickrobot, 11 links, 10 joints
Links:
- added link lidar_link, mass 0.2; visual mesh filename=/home/mickrobot/ros2_mick_ws/src/mick_robot/mickrobot_descr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 scale=0.001 0.001 0.001
- link base_link: geometry collision box size=0.6 0.333 0.16; visual mesh filename=/home/mickrobot/ros2_mick_ws/src/mick_robot/mickrobot_descr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 scale=0.001 0.001 0.001
- link left_back_wheel: geometry collision cylinder length=0.06 radius=0.1016; visual mesh filename=/home/mickrobot/ros2_mick_ws/src/mick_robot/mickrobot_descr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 scale=0.001 0.001 0.001
- link left_front_wheel: geometry collision cylinder length=0.06 radius=0.1016; visual mesh filename=/home/mickrobot/ros2_mick_ws/src/mick_robot/mickrobot_descr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 scale=0.001 0.001 0.001
- link right_back_wheel: geometry collision cylinder length=0.06 radius=0.1016; visual mesh filename=/home/mickrobot/ros2_mick_ws/src/mick_robot/mickrobot_descr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 scale=0.001 0.001 0.001
- link right_front_wheel: geometry collision cylinder length=0.06 radius=0.1016; visual mesh filename=/home/mickrobot/ros2_mick_ws/src/mick_robot/mickrobot_descr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 scale=0.001 0.001 0.001
- link sensor_link: geometry collision box size=0.09 0.12 0.20; visual mesh filename=/home/mickrobot/ros2_mick_ws/src/mick_robot/mickrobot_descr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 scale=0.001 0.001 0.001
Joints:
- added joint lidar_joint: type fixed, parent base_link, child lidar_link, origin xyz=0.23 0.0 0.40, axis 0 0 1, limit effort=0 velocity=0

File: mickrobot_description/urdf/mickrobot_stl_rviz.urdf (robot description, URDF)
Before this commit: robot mickrobot, 11 links, 10 joints
Links:
- added link lidar_link, mass 0.2; visual mesh filename=package://mickrobot_description/urdf/mesh/lidar.STL scale=0.001 0.001 0.001
Joints:
- added joint lidar_joint: type fixed, parent base_link, child lidar_link, origin xyz=0.23 0.0 0.40, axis 0 0 1, limit effort=0 velocity=0
- joint left_back_wheel_joint: type continuous -> fixed
- joint left_front_wheel_joint: type continuous -> fixed
- joint right_back_wheel_joint: type continuous -> fixed
- joint right_front_wheel_joint: type continuous -> fixed
